File: caitlinV3-christmas-ornament.kicad_pcb (KiCad board)
At the start: 2 copper layers, 66 x 106.7 mm, 35 parts

Commit message: Created images folder
Other:
- board text removed: "This work is licensed under a Creative Commons Attribution 4.0 International License."
Changed lines of the file:
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@@
   (general
     (thickness 1.6)
-    (drawings 38)
+    (drawings 37)
     (tracks 20)
     (zones 0)
@@
     )
   )
-  (gr_text "This work is licensed under a Creative Commons Attribution 4.0 International License." (at 231.14 176.53) (layer F.Cu)
-    (effects (font (size 1.5 1.5) (thickness 0.3)))
-  )
   (gr_text "CaitlinV3\nX-MAS TREE\n2019" (at 152.4 93.98) (layer F.SilkS)
